Commit message: fixed gmapping files & fxing converter issues

File: urdf/vaccumbot_camera.xacro (robot description, xacro)
@@ -16,5 +16,5 @@
     <sensor type="camera" name="camera">
     <pose> 0 0 0 0 0 0 </pose>
-    <visualize>true</visualize>
+    <visualize>false</visualize>
     <update_rate>10.0</update_rate>
     <camera>

File: urdf/vaccumbot_gazebo_control.xacro (robot description, xacro)
@@ -30,5 +30,5 @@
   <!-- GAZEBO MATERIAL -->
   <gazebo reference="chassis_link">
-      <material>Gazebo/Orange</material>
+      <material>Gazebo/Black</material>
   </gazebo>
   <gazebo reference="lw_link">
