Commit message: added gmapping files & sensor fix under progress

File: urdf/vaccumbot.urdf.xacro (robot description, xacro)
@@ -3,6 +3,6 @@
   <xacro:include filename="$(find vaccumbot)/urdf/vaccumbot_core.xacro" />
   <xacro:include filename="$(find vaccumbot)/urdf/vaccumbot_gazebo_control.xacro" />
-  <!-- <xacro:include filename="$(find vaccumbot)/urdf/vaccumbot_camera.xacro" /> -->
-  <!-- <xacro:include filename="$(find vaccumbot)/urdf/vaccumbot_depth_camera.xacro" /> -->
+  <xacro:include filename="$(find vaccumbot)/urdf/vaccumbot_camera.xacro" />
+  <xacro:include filename="$(find vaccumbot)/urdf/vaccumbot_depth_camera.xacro" />
   <xacro:include filename="$(find vaccumbot)/urdf/vaccumbot_lidar.xacro" />
 </robot>

File: urdf/vaccumbot_core.xacro (robot description, xacro)
@@ -486,5 +486,6 @@
     <origin
       xyz="0.11856 0 0.12179"
-      rpy="0 -0.17453 0" />
+      rpy="0 0 0" />
+    <!-- use this value for pitch -0.17453 -->
     <parent
       link="base_link" />

File: urdf/vaccumbot_lidar.xacro (robot description, xacro)
@@ -6,12 +6,12 @@
   </gazebo>
   <!-- DEPTH CAMERA OPTICAL LINK-->
-  <joint name="depcam_opt" type="fixed">
+  <joint name="laser_opt" type="fixed">
     <parent link="tcam_link"/>
-    <child link="depcam_link_opt"/>
-    <origin xyz="0 0 0" rpy="-1.57 0 -1.57"/>
+    <child link="laser_link_opt"/>
+    <origin xyz="0 0 0" rpy="0 0 0"/>
   </joint>
-  <link name="depcam_link_opt"></link>
+  <link name="laser_link_opt"></link>
   <!-- DEPTH CAMERA DEFINITION -->
-  <gazebo reference="tcam_link">
+  <gazebo reference="laser_link_opt">
     <sensor name="laser" type="ray">
       <pose> 0 0 0 0 0 0 </pose>
@@ -31,10 +31,8 @@
           </range>
       </ray>
-      <plugin name="laser_controller" filename="libgazebo_ros_ray_sensor.so">
-          <ros>
-              <argument>~/out:=scan</argument>
-          </ros>
-          <output_type>sensor_msgs/LaserScan</output_type>
-          <frame_name>laser_frame</frame_name>
+      <plugin name="laser_controller" filename="libgazebo_ros_laser.so">
+          <topicName>scan</topicName>
+          <!-- <output_type>sensor_msgs/LaserScan</output_type> -->
+          <frame_name>laser_link_opt</frame_name>
       </plugin>
     </sensor>

Commit message: added joint controller and lidar configured for check

File: urdf/vaccumbot.urdf.xacro (robot description, xacro)
@@ -5,4 +5,4 @@
   <xacro:include filename="$(find vaccumbot)/urdf/vaccumbot_camera.xacro" />
   <xacro:include filename="$(find vaccumbot)/urdf/vaccumbot_depth_camera.xacro" />
-  <!-- <xacro:include filename="$(find vaccumbot)/urdf/vaccumbot_lidar.xacro" /> -->
+  <xacro:include filename="$(find vaccumbot)/urdf/vaccumbot_lidar.xacro" />
 </robot>

File: urdf/vaccumbot_depth_camera.xacro (robot description, xacro)
@@ -17,11 +17,11 @@
       <pose> 0 0 0 0 0 0 </pose>
       <visualize>true</visualize>
-      <update_rate>10</update_rate>
+      <update_rate>20</update_rate>
       <camera>
           <horizontal_fov>1.089</horizontal_fov>
           <image>
               <format>B8G8R8</format>
-              <width>640</width>
-              <height>480</height>
+              <width>800</width>
+              <height>800</height>
           </image>
           <clip>
@@ -41,5 +41,5 @@
           <pointCloudTopicName>/camera1/depth/points</pointCloudTopicName>
           <min_depth>0.1</min_depth>
-          <max_depth>100.0</max_depth>
+          <max_depth>200.0</max_depth>
       </plugin>
     </sensor>

File: urdf/vaccumbot_gazebo_control.xacro (robot description, xacro)
@@ -1,4 +1,27 @@
 <?xml version="1.0"?>
 <robot name="vaccumbot" xmlns:xacro="http://www.ros.org/wiki/xacro">
+  <gazebo>
+    <plugin name="gazebo_ros_control" filename="libgazebo_ros_control.so"/>
+  </gazebo>
+  <transmission name="rvc_link_trans">
+    <type>transmission_interface/SimpleTransmission</type>
+    <joint name="rvc">
+    <hardwareInterface>hardware_interface/EffortJointInterface</hardwareInterface>
+    </joint>
+    <actuator name="rvc_link_trans">
+    <hardwareInterface>hardware_interface/EffortJointInterface</hardwareInterface>
+      <mechanicalReduction>1</mechanicalReduction>
+    </actuator>
+  </transmission>
+  <transmission name="fvc_link_trans">
+    <type>transmission_interface/SimpleTransmission</type>
+    <joint name="fvc">
+    <hardwareInterface>hardware_interface/EffortJointInterface</hardwareInterface>
+    </joint>
+    <actuator name="fvc_link_trans">
+    <hardwareInterface>hardware_interface/EffortJointInterface</hardwareInterface>
+      <mechanicalReduction>1</mechanicalReduction>
+    </actuator>
+  </transmission>
   <!-- DIFFERENTIAL CONTROL -->
   <gazebo>

File: urdf/vaccumbot_lidar.xacro (robot description, xacro)
@@ -32,5 +32,5 @@
       </ray>
       <plugin name="laser_controller" filename="libgazebo_ros_laser.so">
-          <topicName>scan</topicName>
+          <topicName>/laser/scan</topicName>
           <!-- <output_type>sensor_msgs/LaserScan</output_type> -->
           <frameName>laser_link_opt</frameName>
